File: hardware/common_PCB/FRC_5690_Common_PCB/FRC_5690_Common_PCB.kicad_pcb (KiCad board)
At the start: 2 copper layers, 74.8 x 78.6 mm, 41 parts, among them J1 5V in, J10 UART, J11 LED 0, J12 LED 1, J13 Analog In, J14 Micro_SD_Card, J15 CONFIG, J17 Conn_01x03_Pin, J18 Conn_01x03_Pin, J19 Conn_01x03_Pin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

Commit message: update pcb
Parts:
- added J16: GND, Connector_PinHeader_2.54mm:PinHeader_1x03_P2.54mm_Vertical, F.Cu at (166.5, 95.6)
- J9: value SPI1-1 -> SPI 1
- moved J13 3.31 mm to (162.6, 95.6)
- moved Q1 2.99 mm to (150.5, 94.0)
- moved R4 1.67 mm to (156.2, 92.1)
Routing:
- net +5V: track 119.7 -> 121.8 mm
- net Net-(D2-DIN): track 10.9 -> 13.0 mm
- net Net-(Q1-B): track 2.54 -> 4.56 mm
- net /RGB_LED1: track 10.1 -> 8.53 mm
- net /ADC1: track 25.6 -> 24.6 mm
