File: hardware/common_PCB/FRC_5690_Common_PCB/FRC_5690_Common_PCB.kicad_sch (KiCad schematic)
At the start: 41 parts, among them J1 5V in, J10 UART, J11 LED 0, J12 LED 1, J13 Analog In, J14 Micro_SD_Card, J15 CONFIG, J17 Conn_01x03_Pin, J18 Conn_01x03_Pin, J19 Conn_01x03_Pin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

Commit message: update pcb
Parts:
- added J16: GND, Connector_PinHeader_2.54mm:PinHeader_1x03_P2.54mm_Vertical, symbol Connector:Conn_01x03_Pin
Connections:
- net GND: now also J16.1 (Pin_1), J16.2 (Pin_2), J16.3 (Pin_3)
Changed lines of the file:
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@@
   (junction (at 88.9 73.66) (diameter 0) (color 0 0 0 0)
   )
+  (junction (at 191.77 100.33) (diameter 0) (color 0 0 0 0)
+  )
   (junction (at 222.25 149.86) (diameter 0) (color 0 0 0 0)
   )
@@
   )
   (junction (at 88.9 68.58) (diameter 0) (color 0 0 0 0)
+  )
+  (junction (at 191.77 102.87) (diameter 0) (color 0 0 0 0)
   )
   (junction (at 224.79 63.5) (diameter 0) (color 0 0 0 0)
@@
     (stroke (width 0) (type default))
   )
+  (wire (pts (xy 191.77 100.33) (xy 191.77 102.87))
+    (stroke (width 0) (type default))
+  )
   (wire (pts (xy 59.69 162.56) (xy 68.58 162.56))
     (stroke (width 0) (type default))
@@
     (stroke (width 0) (type default))
   )
+  (wire (pts (xy 191.77 97.79) (xy 191.77 100.33))
+    (stroke (width 0) (type default))
+  )
   (wire (pts (xy 119.38 97.79) (xy 129.54 97.79))
     (stroke (width 0) (type default))
@@
   )
   (wire (pts (xy 224.79 93.98) (xy 232.41 93.98))
+    (stroke (width 0) (type default))
+  )
+  (wire (pts (xy 191.77 102.87) (xy 191.77 106.68))
     (stroke (width 0) (type default))
   )
@@
         (path "/61912a13-ede8-48b1-a32d-9390036060d9"
           (reference "#PWR05") (unit 1)
+        )
+      )
+    )
+  )
+  (symbol (lib_id "power:GND") (at 191.77 106.68 0) (unit 1)
+    (in_bom yes) (on_board yes) (dnp no) (fields_autoplaced)
+    (property "Reference" "#PWR061" (at 191.77 113.03 0)
+      (effects (font (size 1.27 1.27)) hide)
+    )
+    (property "Value" "GND" (at 191.77 111.76 0)
+      (effects (font (size 1.27 1.27)))
+    )
+    (property "Footprint" "" (at 191.77 106.68 0)
+      (effects (font (size 1.27 1.27)) hide)
+    )
+    (property "Datasheet" "" (at 191.77 106.68 0)
+      (effects (font (size 1.27 1.27)) hide)
+    )
+    (pin "1")
+    (instances
+      (project "FRC_5690_Common_PCB"
+        (path "/61912a13-ede8-48b1-a32d-9390036060d9"
+          (reference "#PWR061") (unit 1)
         )
       )
@@
         )
       )
+    )
+  )
+  (symbol (lib_id "Connector:Conn_01x03_Pin") (at 196.85 100.33 180) (unit 1)
+    (in_bom yes) (on_board yes) (dnp no) (fields_autoplaced)
+    (property "Reference" "J16" (at 198.12 99.695 0)
+      (effects (font (size 1.27 1.27)) (justify right))
+    )
+    (property "Value" "GND" (at 198.12 102.235 0)
+      (effects (font (size 1.27 1.27)) (justify right))
+    )
+    (property "Footprint" "Connector_PinHeader_2.54mm:PinHeader_1x03_P2.54mm_Vertical" (at 196.85 100.33 0)
+      (effects (font (size 1.27 1.27)) hide)
+    )
+    (property "Datasheet" "~" (at 196.85 100.33 0)
+      (effects (font (size 1.27 1.27)) hide)
+    )
+    (pin "1")
+    (pin "2")
+    (pin "3")
+    (instances
+      (project "FRC_5690_Common_PCB"
+        (path "/61912a13-ede8-48b1-a32d-9390036060d9"
+          (reference "J16") (unit 1)
+        )
+      )
