File: hardware/common_PCB/ConnectorX/ConnectorX.kicad_pcb (KiCad board)
At the start: 2 copper layers, 79 x 94.7 mm, 41 parts, among them J1 Barrel_Jack_Switch, J10 I2C 1, J11 SPI 0, J2 Conn_01x03_Socket, J3 Conn_01x03_Socket, J4 Conn_01x03_Socket, J5 Conn_01x03_Socket, J6 Conn_01x03_Socket, J7 RIO side, J8 Top side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

Commit message: Finalize ConnectorX
Parts:
- Q1: value IRLML5203 -> IRLML5203TRPBF
Changed lines of the file:
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@@
       (outputformat 1)
       (mirror false)
-      (drillshape 1)
+      (drillshape 0)
       (scaleselection 1)
-      (outputdirectory "")
+      (outputdirectory "ConnectorX-gerbers/")
     )
   )
@@
     (fp_line (start 4.11 2.7) (end 3.11 2.7)
       (stroke (width 0.1) (type solid)) (layer "F.Fab"))
-    (pad "1" smd roundrect (at -5.04 -2.28) (size 2.2 1.2) (layers "F.Cu" "F.Paste" "F.Mask") (roundrect_rratio 0.208333)
+    (pad "1" smd roundrect (at -5.04 -2.28) (size 2.2 1.2) (layers "F.Cu" "F.Paste" "F.Mask") (roundrect_rratio 0.2083333333)
       (net 1 "+5V") (pinfunction "K") (pintype "passive"))
-    (pad "2" smd roundrect (at -0.415 -1.525) (size 3.05 2.75) (layers "F.Cu" "F.Paste") (roundrect_rratio 0.090909)
+    (pad "2" smd roundrect (at -0.415 -1.525) (size 3.05 2.75) (layers "F.Cu" "F.Paste") (roundrect_rratio 0.09090909091)
       (net 6 "Net-(D1-A)") (pinfunction "A") (pintype "passive"))
-    (pad "2" smd roundrect (at -0.415 1.525) (size 3.05 2.75) (layers "F.Cu" "F.Paste") (roundrect_rratio 0.090909)
+    (pad "2" smd roundrect (at -0.415 1.525) (size 3.05 2.75) (layers "F.Cu" "F.Paste") (roundrect_rratio 0.09090909091)
       (net 6 "Net-(D1-A)") (pinfunction "A") (pintype "passive"))
-    (pad "2" smd roundrect (at 1.26 0) (size 6.4 5.8) (layers "F.Cu" "F.Mask") (roundrect_rratio 0.043103)
+    (pad "2" smd roundrect (at 1.26 0) (size 6.4 5.8) (layers "F.Cu" "F.Mask") (roundrect_rratio 0.04310293103)
       (net 6 "Net-(D1-A)") (pinfunction "A") (pintype "passive"))
-    (pad "2" smd roundrect (at 2.935 -1.525) (size 3.05 2.75) (layers "F.Cu" "F.Paste") (roundrect_rratio 0.090909)
+    (pad "2" smd roundrect (at 2.935 -1.525) (size 3.05 2.75) (layers "F.Cu" "F.Paste") (roundrect_rratio 0.09090909091)
       (net 6 "Net-(D1-A)") (pinfunction "A") (pintype "passive"))
-    (pad "2" smd roundrect (at 2.935 1.525) (size 3.05 2.75) (layers "F.Cu" "F.Paste") (roundrect_rratio 0.090909)
+    (pad "2" smd roundrect (at 2.935 1.525) (size 3.05 2.75) (layers "F.Cu" "F.Paste") (roundrect_rratio 0.09090909091)
       (net 6 "Net-(D1-A)") (pinfunction "A") (pintype "passive"))
-    (pad "3" smd roundrect (at -5.04 2.28) (size 2.2 1.2) (layers "F.Cu" "F.Paste" "F.Mask") (roundrect_rratio 0.208333))
+    (pad "3" smd roundrect (at -5.04 2.28) (size 2.2 1.2) (layers "F.Cu" "F.Paste" "F.Mask") (roundrect_rratio 0.2083333333))
     (model "${KICAD6_3DMODEL_DIR}/Package_TO_SOT_SMD.3dshapes/TO-252-2.wrl"
       (offset (xyz 0 0 0))
@@
     (fp_line (start 9.87 7.2) (end 8.82 7.2)
       (stroke (width 0.1) (type solid)) (layer "F.Fab"))
-    (pad "1" thru_hole roundrect (at 0 0 90) (size 2.7 2.7) (drill 1.7) (layers "*.Cu" "*.Mask") (roundrect_rratio 0.092593)
+    (pad "1" thru_hole roundrect (at 0 0 90) (size 2.7 2.7) (drill 1.7) (layers "*.Cu" "*.Mask") (roundrect_rratio 0.09259296296)
       (net 4 "Net-(D5-VDD)") (pinfunction "Pin_1") (pintype "passive"))
     (pad "2" thru_hole circle (at 3.96 0 90) (size 2.7 2.7) (drill 1.7) (layers "*.Cu" "*.Mask")
@@
     (fp_line (start 9.87 7.2) (end 8.82 7.2)
       (stroke (width 0.1) (type solid)) (layer "F.Fab"))
-    (pad "1" thru_hole roundrect (at 0 0 90) (size 2.7 2.7) (drill 1.7) (layers "*.Cu" "*.Mask") (roundrect_rratio 0.092593)
+    (pad "1" thru_hole roundrect (at 0 0 90) (size 2.7 2.7) (drill 1.7) (layers "*.Cu" "*.Mask") (roundrect_rratio 0.09259296296)
       (net 5 "Net-(D6-VDD)") (pinfunction "Pin_1") (pintype "passive"))
     (pad "2" thru_hole circle (at 3.96 0 90) (size 2.7 2.7) (drill 1.7) (layers "*.Cu" "*.Mask")
@@
         (effects (font (size 1 1) (thickness 0.15)))
     )
-    (fp_text value "IRLML5203" (at 0 2.4 90) (layer "F.Fab")
+    (fp_text value "IRLML5203TRPBF" (at 2 2.6 90) (layer "F.Fab")
         (effects (font (size 1 1) (thickness 0.15)))
     )
@@
   )
   (gr_text_box "Base address = 0010000 = 0x10\nToggle last three bits with switch\nMax address = 0x17"
-    (start 145.6 50) (end 157 55.2) (layer "F.SilkS")
-      (effects (font (size 0.508 0.508) (thickness 0.0635)) (justify left top))
+    (start 139.85 48.2) (end 155.35 55.6) (layer "F.SilkS")
+      (effects (font (size 0.7112 0.7112) (thickness 0.0635)) (justify left top))
     (stroke (width 0.15) (type dash))  )
   (gr_text_box "Status indicators"
@@
       (effects (font (size 1 1) (thickness 0.15)) (justify left top))
     (stroke (width 0.15) (type dot))  )
-  (gr_text_box "For config mode:\nHold CONFIG\nPress RESET\nRelease CONFIG\nBlue CONFIG LED should illuminate"
-    (start 125.8 47.5) (end 119.8 56.9) (angle 270) (layer "F.SilkS")
-      (effects (font (size 0.508 0.508) (thickness 0.0635)) (justify left top))
+  (gr_text_box "For config mode:\nHold CONFIG\nPress RESET\nBlue CONFIG LED should illuminate\nRelease CONFIG"
+    (start 127.2 47.7) (end 118.2 57.1) (angle 270) (layer "F.SilkS")
+      (effects (font (size 0.635 0.635) (thickness 0.0635)) (justify left top))
     (stroke (width 0.15) (type dash))  )
   (segment (start 167.9 67.1) (end 167.9 62.75) (width 0.3048) (layer "F.Cu") (net 1))
